Commit message: update

File: src/ur5_3f/ur5_3f_description/urdf/UR5_3f_macro.xacro (robot description, xacro)
@@ -1,17 +1,24 @@
 <?xml version="1.0"?>
-<robot xmlns:xacro="http://ros.org/wiki/xacro"
-	name="UR5_3f">
-	<xacro:arg name="limited" default="true"/>
-	<!-- UR from ROS industrial repos -->
-	<xacro:include filename="$(find ur_description)/urdf/ur5_robot.urdf.xacro"/>
-	<xacro:ur5_robot prefix="simple_arm_" joint_limited="false"/>
-	<!-- Robotiq from ROS industrial repos -->
-	<xacro:include filename="$(find robotiq_3f_gripper_visualization)/cfg/robotiq_hand_macro.urdf.xacro"/>
-	<xacro:robotiq_hand prefix="simple_gripper_" reflect="1" parent="simple_arm_tool0">
-		<origin xyz="0 0 0" rpy="${pi/2} ${pi/2} 0"/>
-	</xacro:robotiq_hand>
-	<gazebo>
-		<plugin name="gazebo_ros_control" filename="libgazebo_ros_control.so">
-		</plugin>
-	</gazebo>
+<robot xmlns:xacro="http://wiki.ros.org/xacro"
+       name="ur5" >
+  <xacro:arg name="transmission_hw_interface" default="hardware_interface/PositionJointInterface"/>
+  <!-- common stuff -->
+  <xacro:include filename="$(find ur_description)/urdf/common.gazebo.xacro" />
+  <!-- ur5 -->
+  <xacro:include filename="$(find ur_description)/urdf/ur5.urdf.xacro" />
+  <!-- arm -->
+  <xacro:ur5_robot prefix="" joint_limited="false"
+    transmission_hw_interface="$(arg transmission_hw_interface)"
+  />
+  <!-- Robotiq from ROS industrial repos -->
+    <xacro:include filename="$(find robotiq_3f_gripper_visualization)/cfg/robotiq_hand_macro.urdf.xacro"/>
+    <xacro:robotiq_hand prefix="r3f_" reflect="1" parent="tool0">
+      <origin xyz="0 0 0.05" rpy="${pi/2} 0 0"/>
+    </xacro:robotiq_hand>
+  <link name="world" />
+  <joint name="world_joint" type="fixed">
+    <parent link="world" />
+    <child link = "base_link" />
+    <origin xyz="0.0 0.0 0.0" rpy="0.0 0.0 0.0" />
+  </joint>
 </robot>

Commit message: switched robotiq repos, trying to make it work

File: src/ur5_3f/ur5_3f_description/urdf/UR5_3f_macro.xacro (robot description, xacro)
@@ -1,5 +1,5 @@
 <?xml version="1.0"?>
 <robot xmlns:xacro="http://wiki.ros.org/xacro"
-       name="ur5" >
+       name="ur5_3f" >
   <xacro:arg name="transmission_hw_interface" default="hardware_interface/PositionJointInterface"/>
   <!-- common stuff -->
@@ -13,9 +13,9 @@
   <!-- Robotiq from ROS industrial repos -->
     <xacro:include filename="$(find robotiq_3f_gripper_visualization)/cfg/robotiq_hand_macro.urdf.xacro"/>
-    <xacro:robotiq_hand prefix="r3f_" reflect="1" parent="tool0">
-      <origin xyz="0 0 0.05" rpy="${pi/2} 0 0"/>
+    <xacro:robotiq_hand prefix="r3f_" reflect="" parent="tool0">
+      <origin xyz="0 0 0.1" rpy="${pi/2} 0 0"/>
     </xacro:robotiq_hand>
-    <xacro:include filename="$(find ur5_3f)/ur5_3f_description/urdf/robotiq_3f_gripper.transmission.xacro"/>
-    <xacro:robotiq_3f_gripper_transmission prefix="r3f_"/>
+   <!-- <xacro:include filename="$(find ur5_3f)/ur5_3f_description/urdf/robotiq_3f_gripper.transmission.xacro"/>
+    <xacro:robotiq_3f_gripper_transmission prefix="r3f_"/>-->
   <link name="world" />
   <joint name="world_joint" type="fixed">
@@ -24,3 +24,15 @@
     <origin xyz="0.0 0.0 0.0" rpy="0.0 0.0 0.0" />
   </joint>
+    <gazebo>
+    <!-- plugin for the RobotiQ hand -->
+    <plugin name="robotiq_hand_plugin" filename="libRobotiqHandPlugin.so">
+      <kp_position>10.0</kp_position>
+      <kd_position>0.5</kd_position>
+      <!-- Some optional parameters. Check the plugin header file for all of them. -->
+      <prefix>r3f_</prefix>
+      <!-- This is chosen, so it's compatible with the "Robotiq3FGripperSimpleController.py"-->
+      <topic_command>/Robotiq3FGripperRobotOutput</topic_command>
+      <!-- <topic_state>/hand/state</topic_state> -->
+    </plugin>
+  </gazebo>
 </robot>

File: src/ur5_3f/ur5_3f_description/urdf/UR5_3f_macro.xacro.urdf (robot description, URDF)
Before this commit: robot ur5, 51 links, 50 joints
Joints:
- joint r3f_robotiq_hand_joint: origin xyz=0 0 0.05 rpy=1.57079632679 0 0 -> xyz=0 0 0.1 rpy=1.57079632679 0 0

Commit message: updates

File: src/ur5_3f/ur5_3f_description/urdf/UR5_3f_macro.xacro (robot description, xacro)
@@ -14,5 +14,5 @@
     <xacro:include filename="$(find robotiq_3f_gripper_visualization)/cfg/robotiq_hand_macro.urdf.xacro"/>
     <xacro:robotiq_hand prefix="r3f_" reflect="" parent="tool0">
-      <origin xyz="0 0 0.1" rpy="${pi/2} 0 0"/>
+      <origin xyz="0 0 0.055" rpy="${pi/2} 0 0"/>
     </xacro:robotiq_hand>
    <!-- <xacro:include filename="$(find ur5_3f)/ur5_3f_description/urdf/robotiq_3f_gripper.transmission.xacro"/>

File: src/ur5_3f/ur5_3f_description/urdf/UR5_3f_macro.xacro.urdf (robot description, URDF)
Before this commit: robot ur5_3f, 51 links, 50 joints
Joints:
- joint r3f_robotiq_hand_joint: origin xyz=0 0 0.1 rpy=1.57079632679 0 0 -> xyz=0 0 0.055 rpy=1.57079632679 0 0

Commit message: attempt

File: src/ur5_3f/ur5_3f_description/urdf/UR5_3f_macro.xacro (robot description, xacro)
@@ -2,5 +2,5 @@
 <robot xmlns:xacro="http://wiki.ros.org/xacro"
        name="ur5_3f" >
-  <xacro:arg name="transmission_hw_interface" default="hardware_interface/PositionJointInterface"/>
+  <xacro:arg name="transmission_hw_interface" default="hardware_interface/EffortJointInterface"/>
   <!-- common stuff -->
   <xacro:include filename="$(find ur_description)/urdf/common.gazebo.xacro" />
@@ -8,11 +8,17 @@
   <xacro:include filename="$(find ur_description)/urdf/ur5.urdf.xacro" />
   <!-- arm -->
-  <xacro:ur5_robot prefix="" joint_limited="false"
+  <xacro:ur5_robot prefix="ur5_" joint_limited="false"
     transmission_hw_interface="$(arg transmission_hw_interface)"
   />
+<!--  <link name="hand_anchor_link"/>
+  <joint name="hand_anchor_joint" type="fixed">
+    <parent link="base_link" />
+    <child link = "hand_anchor_link" />
+    <origin xyz="0.0 1.0 0.0" rpy="0.0 0.0 0.0" />
+  </joint>-->
   <!-- Robotiq from ROS industrial repos -->
     <xacro:include filename="$(find robotiq_3f_gripper_visualization)/cfg/robotiq_hand_macro.urdf.xacro"/>
-    <xacro:robotiq_hand prefix="r3f_" reflect="" parent="tool0">
-      <origin xyz="0 0 0.055" rpy="${pi/2} 0 0"/>
+    <xacro:robotiq_hand prefix="r3f_" reflect="" parent="ur5_shoulder_link">
+      <origin xyz="0 0.4 0.055" rpy="${pi/2} 0 0"/>
     </xacro:robotiq_hand>
    <!-- <xacro:include filename="$(find ur5_3f)/ur5_3f_description/urdf/robotiq_3f_gripper.transmission.xacro"/>
@@ -21,17 +27,14 @@
   <joint name="world_joint" type="fixed">
     <parent link="world" />
-    <child link = "base_link" />
+    <child link = "ur5_base_link" />
     <origin xyz="0.0 0.0 0.0" rpy="0.0 0.0 0.0" />
   </joint>
-    <gazebo>
-    <!-- plugin for the RobotiQ hand -->
+  <!-- plugin for the RobotiQ hand -->
+  <gazebo>
     <plugin name="robotiq_hand_plugin" filename="libRobotiqHandPlugin.so">
       <kp_position>10.0</kp_position>
       <kd_position>0.5</kd_position>
-      <!-- Some optional parameters. Check the plugin header file for all of them. -->
       <prefix>r3f_</prefix>
-      <!-- This is chosen, so it's compatible with the "Robotiq3FGripperSimpleController.py"-->
       <topic_command>/Robotiq3FGripperRobotOutput</topic_command>
-      <!-- <topic_state>/hand/state</topic_state> -->
     </plugin>
   </gazebo>

File: src/ur5_3f/ur5_3f_description/urdf/UR5_3f_macro.xacro.urdf (robot description, URDF)
Before this commit: robot ur5_3f, 51 links, 50 joints
Links:
- removed link base
- removed link base_link
- removed link ee_link
- removed link forearm_link
- removed link shoulder_link
- removed link tool0
- removed link upper_arm_link
- removed link wrist_1_link
- removed link wrist_2_link
- removed link wrist_3_link
- added link ur5_base
- added link ur5_base_link, mass 4.0; collision mesh filename=package://ur_description/meshes/ur5/collision/base.stl; visual mesh filename=package://ur_description/meshes/ur5/visual/base.dae
- added link ur5_ee_link; collision box size=0.01 0.01 0.01
- added link ur5_forearm_link, mass 2.275; collision mesh filename=package://ur_description/meshes/ur5/collision/forearm.stl; visual mesh filename=package://ur_description/meshes/ur5/visual/forearm.dae
- added link ur5_shoulder_link, mass 3.7; collision mesh filename=package://ur_description/meshes/ur5/collision/shoulder.stl; visual mesh filename=package://ur_description/meshes/ur5/visual/shoulder.dae
- added link ur5_tool0
- added link ur5_upper_arm_link, mass 8.393; collision mesh filename=package://ur_description/meshes/ur5/collision/upperarm.stl; visual mesh filename=package://ur_description/meshes/ur5/visual/upperarm.dae
- added link ur5_wrist_1_link, mass 1.219; collision mesh filename=package://ur_description/meshes/ur5/collision/wrist1.stl; visual mesh filename=package://ur_description/meshes/ur5/visual/wrist1.dae
- added link ur5_wrist_2_link, mass 1.219; collision mesh filename=package://ur_description/meshes/ur5/collision/wrist2.stl; visual mesh filename=package://ur_description/meshes/ur5/visual/wrist2.dae
- added link ur5_wrist_3_link, mass 0.1879; collision mesh filename=package://ur_description/meshes/ur5/collision/wrist3.stl; visual mesh filename=package://ur_description/meshes/ur5/visual/wrist3.dae
Joints:
- removed joint base_link-base_fixed_joint
- removed joint ee_fixed_joint
- removed joint elbow_joint
- removed joint shoulder_lift_joint
- removed joint shoulder_pan_joint
- removed joint wrist_1_joint
- removed joint wrist_2_joint
- removed joint wrist_3_joint
- removed joint wrist_3_link-tool0_fixed_joint
- added joint ur5_base_link-base_fixed_joint: type fixed, parent ur5_base_link, child ur5_base, origin xyz=0 0 0 rpy=0 0 -3.14159265359
- added joint ur5_ee_fixed_joint: type fixed, parent ur5_wrist_3_link, child ur5_ee_link, origin xyz=0.0 0.0823 0.0 rpy=0.0 0.0 1.57079632679
- added joint ur5_elbow_joint: type revolute, parent ur5_upper_arm_link, child ur5_forearm_link, origin xyz=0.0 -0.1197 0.425 rpy=0.0 0.0 0.0, axis 0 1 0, limit lower=-3.14159265359 upper=3.14159265359 effort=150.0 velocity=3.15
- added joint ur5_shoulder_lift_joint: type revolute, parent ur5_shoulder_link, child ur5_upper_arm_link, origin xyz=0.0 0.13585 0.0 rpy=0.0 1.57079632679 0.0, axis 0 1 0, limit lower=-6.28318530718 upper=6.28318530718 effort=150.0 velocity=3.15
- added joint ur5_shoulder_pan_joint: type revolute, parent ur5_base_link, child ur5_shoulder_link, origin xyz=0.0 0.0 0.089159 rpy=0.0 0.0 0.0, axis 0 0 1, limit lower=-6.28318530718 upper=6.28318530718 effort=150.0 velocity=3.15
- added joint ur5_wrist_1_joint: type revolute, parent ur5_forearm_link, child ur5_wrist_1_link, origin xyz=0.0 0.0 0.39225 rpy=0.0 1.57079632679 0.0, axis 0 1 0, limit lower=-6.28318530718 upper=6.28318530718 effort=28.0 velocity=3.2
- added joint ur5_wrist_2_joint: type revolute, parent ur5_wrist_1_link, child ur5_wrist_2_link, origin xyz=0.0 0.093 0.0 rpy=0.0 0.0 0.0, axis 0 0 1, limit lower=-6.28318530718 upper=6.28318530718 effort=28.0 velocity=3.2
- added joint ur5_wrist_3_joint: type revolute, parent ur5_wrist_2_link, child ur5_wrist_3_link, origin xyz=0.0 0.0 0.09465 rpy=0.0 0.0 0.0, axis 0 1 0, limit lower=-6.28318530718 upper=6.28318530718 effort=28.0 velocity=3.2
- added joint ur5_wrist_3_link-tool0_fixed_joint: type fixed, parent ur5_wrist_3_link, child ur5_tool0, origin xyz=0 0.0823 0 rpy=-1.57079632679 0 0
- joint r3f_robotiq_hand_joint: origin xyz=0 0 0.055 rpy=1.57079632679 0 0 -> xyz=0 0.4 0.055 rpy=1.57079632679 0 0; parent tool0 -> ur5_shoulder_link
- joint world_joint: child base_link -> ur5_base_link

Commit message: RADI

File: src/ur5_3f/ur5_3f_description/urdf/UR5_3f_macro.xacro (robot description, xacro)
@@ -4,9 +4,9 @@
   <xacro:arg name="transmission_hw_interface" default="hardware_interface/EffortJointInterface"/>
   <!-- common stuff -->
-  <xacro:include filename="$(find ur_description)/urdf/common.gazebo.xacro" />
+  <xacro:include filename="$(find ur5_3f)/ur5_3f_description/urdf/common.gazebo.xacro" />
   <!-- ur5 -->
-  <xacro:include filename="$(find ur_description)/urdf/ur5.urdf.xacro" />
+  <xacro:include filename="$(find ur5_3f)/ur5_3f_description/urdf/ur5.urdf.xacro" />
   <!-- arm -->
-  <xacro:ur5_robot prefix="ur5_" joint_limited="false"
+  <xacro:ur5_robot prefix="" joint_limited="false"
     transmission_hw_interface="$(arg transmission_hw_interface)"
   />
@@ -19,6 +19,6 @@
   <!-- Robotiq from ROS industrial repos -->
     <xacro:include filename="$(find robotiq_3f_gripper_visualization)/cfg/robotiq_hand_macro.urdf.xacro"/>
-    <xacro:robotiq_hand prefix="r3f_" reflect="" parent="ur5_shoulder_link">
-      <origin xyz="0 0.4 0.055" rpy="${pi/2} 0 0"/>
+    <xacro:robotiq_hand prefix="r3f_" reflect="" parent="tool0">
+      <origin xyz="0 0 0.055" rpy="${pi/2} 0 0"/>
     </xacro:robotiq_hand>
    <!-- <xacro:include filename="$(find ur5_3f)/ur5_3f_description/urdf/robotiq_3f_gripper.transmission.xacro"/>
@@ -27,5 +27,5 @@
   <joint name="world_joint" type="fixed">
     <parent link="world" />
-    <child link = "ur5_base_link" />
+    <child link = "base_link" />
     <origin xyz="0.0 0.0 0.0" rpy="0.0 0.0 0.0" />
   </joint>

File: src/ur5_3f/ur5_3f_description/urdf/UR5_3f_macro.xacro.urdf (robot description, URDF)
Before this commit: robot ur5_3f, 51 links, 50 joints
Links:
- removed link ur5_base
- removed link ur5_base_link
- removed link ur5_ee_link
- removed link ur5_forearm_link
- removed link ur5_shoulder_link
- removed link ur5_tool0
- removed link ur5_upper_arm_link
- removed link ur5_wrist_1_link
- removed link ur5_wrist_2_link
- removed link ur5_wrist_3_link
- added link base
- added link base_link, mass 4.0; collision mesh filename=package://ur_description/meshes/ur5/collision/base.stl; visual mesh filename=package://ur_description/meshes/ur5/visual/base.dae
- added link ee_link; collision box size=0.01 0.01 0.01
- added link forearm_link, mass 2.275; collision mesh filename=package://ur_description/meshes/ur5/collision/forearm.stl; visual mesh filename=package://ur_description/meshes/ur5/visual/forearm.dae
- added link shoulder_link, mass 3.7; collision mesh filename=package://ur_description/meshes/ur5/collision/shoulder.stl; visual mesh filename=package://ur_description/meshes/ur5/visual/shoulder.dae
- added link tool0
- added link upper_arm_link, mass 8.393; collision mesh filename=package://ur_description/meshes/ur5/collision/upperarm.stl; visual mesh filename=package://ur_description/meshes/ur5/visual/upperarm.dae
- added link wrist_1_link, mass 1.219; collision mesh filename=package://ur_description/meshes/ur5/collision/wrist1.stl; visual mesh filename=package://ur_description/meshes/ur5/visual/wrist1.dae
- added link wrist_2_link, mass 1.219; collision mesh filename=package://ur_description/meshes/ur5/collision/wrist2.stl; visual mesh filename=package://ur_description/meshes/ur5/visual/wrist2.dae
- added link wrist_3_link, mass 0.1879; collision mesh filename=package://ur_description/meshes/ur5/collision/wrist3.stl; visual mesh filename=package://ur_description/meshes/ur5/visual/wrist3.dae
Joints:
- removed joint ur5_base_link-base_fixed_joint
- removed joint ur5_ee_fixed_joint
- removed joint ur5_elbow_joint
- removed joint ur5_shoulder_lift_joint
- removed joint ur5_shoulder_pan_joint
- removed joint ur5_wrist_1_joint
- removed joint ur5_wrist_2_joint
- removed joint ur5_wrist_3_joint
- removed joint ur5_wrist_3_link-tool0_fixed_joint
- added joint base_link-base_fixed_joint: type fixed, parent base_link, child base, origin xyz=0 0 0 rpy=0 0 -3.14159265359
- added joint ee_fixed_joint: type fixed, parent wrist_3_link, child ee_link, origin xyz=0.0 0.0823 0.0 rpy=0.0 0.0 1.57079632679
- added joint elbow_joint: type revolute, parent upper_arm_link, child forearm_link, origin xyz=0.0 -0.1197 0.425 rpy=0.0 0.0 0.0, axis 0 1 0, limit lower=-3.14159265359 upper=3.14159265359 effort=150.0 velocity=3.15
- added joint shoulder_lift_joint: type revolute, parent shoulder_link, child upper_arm_link, origin xyz=0.0 0.13585 0.0 rpy=0.0 1.57079632679 0.0, axis 0 1 0, limit lower=-6.28318530718 upper=6.28318530718 effort=150.0 velocity=3.15
- added joint shoulder_pan_joint: type revolute, parent base_link, child shoulder_link, origin xyz=0.0 0.0 0.089159 rpy=0.0 0.0 0.0, axis 0 0 1, limit lower=-6.28318530718 upper=6.28318530718 effort=150.0 velocity=3.15
- added joint wrist_1_joint: type revolute, parent forearm_link, child wrist_1_link, origin xyz=0.0 0.0 0.39225 rpy=0.0 1.57079632679 0.0, axis 0 1 0, limit lower=-6.28318530718 upper=6.28318530718 effort=28.0 velocity=3.2
- added joint wrist_2_joint: type revolute, parent wrist_1_link, child wrist_2_link, origin xyz=0.0 0.093 0.0 rpy=0.0 0.0 0.0, axis 0 0 1, limit lower=-6.28318530718 upper=6.28318530718 effort=28.0 velocity=3.2
- added joint wrist_3_joint: type revolute, parent wrist_2_link, child wrist_3_link, origin xyz=0.0 0.0 0.09465 rpy=0.0 0.0 0.0, axis 0 1 0, limit lower=-6.28318530718 upper=6.28318530718 effort=28.0 velocity=3.2
- added joint wrist_3_link-tool0_fixed_joint: type fixed, parent wrist_3_link, child tool0, origin xyz=0 0.0823 0 rpy=-1.57079632679 0 0
- joint r3f_robotiq_hand_joint: origin xyz=0 0.4 0.055 rpy=1.57079632679 0 0 -> xyz=0 0 0.055 rpy=1.57079632679 0 0; parent ur5_shoulder_link -> tool0
- joint world_joint: child ur5_base_link -> base_link

Commit message: working simulation

File: src/ur5_3f/ur5_3f_description/urdf/UR5_3f_macro.xacro (robot description, xacro)
@@ -1,20 +1,13 @@
 <?xml version="1.0"?>
 <robot xmlns:xacro="http://wiki.ros.org/xacro"
-       name="ur5_3f" >
+       name="ur5_3f">
   <xacro:arg name="transmission_hw_interface" default="hardware_interface/EffortJointInterface"/>
   <!-- common stuff -->
-  <xacro:include filename="$(find ur5_3f)/ur5_3f_description/urdf/common.gazebo.xacro" />
+  <xacro:include filename="$(find ur5_3f)/ur5_3f_description/urdf/common.gazebo.xacro"/>
   <!-- ur5 -->
-  <xacro:include filename="$(find ur5_3f)/ur5_3f_description/urdf/ur5.urdf.xacro" />
+  <xacro:include filename="$(find ur5_3f)/ur5_3f_description/urdf/ur5.urdf.xacro"/>
   <!-- arm -->
   <xacro:ur5_robot prefix="" joint_limited="false"
-    transmission_hw_interface="$(arg transmission_hw_interface)"
-  />
-<!--  <link name="hand_anchor_link"/>
-  <joint name="hand_anchor_joint" type="fixed">
-    <parent link="base_link" />
-    <child link = "hand_anchor_link" />
-    <origin xyz="0.0 1.0 0.0" rpy="0.0 0.0 0.0" />
-  </joint>-->
+    transmission_hw_interface="$(arg transmission_hw_interface)"/>
   <!-- Robotiq from ROS industrial repos -->
     <xacro:include filename="$(find robotiq_3f_gripper_visualization)/cfg/robotiq_hand_macro.urdf.xacro"/>
@@ -22,6 +15,4 @@
       <origin xyz="0 0 0.055" rpy="${pi/2} 0 0"/>
     </xacro:robotiq_hand>
-   <!-- <xacro:include filename="$(find ur5_3f)/ur5_3f_description/urdf/robotiq_3f_gripper.transmission.xacro"/>
-    <xacro:robotiq_3f_gripper_transmission prefix="r3f_"/>-->
   <link name="world" />
   <joint name="world_joint" type="fixed">
